Commit message: Initia

File: install/mob_rov/share/mob_rov/urdf/mob_rov2.xacro (robot description, xacro)
@@ -57,4 +57,12 @@
   <link name="base_link">
     <!-- Optionally add geometry here -->
+  </link>
+  <!-- BASE_FOOTPRINT LINK -->
+  <joint name="base_footprint_joint" type="fixed">
+      <parent link="base_link"/>
+      <child link="base_footprint"/>
+      <origin xyz="0 0 0" rpy="0 0 0"/>
+  </joint>
+  <link name="base_footprint">
   </link>
   <!-- Chassis link -->
@@ -154,5 +162,6 @@
     <mu2 value="0.001"/>
   </gazebo>
-  <xacro:include filename="gazebo_control.xacro" />
+  <!-- <xacro:include filename="gazebo_control.xacro" /> -->
+  <xacro:include filename="ros2_control.xacro" />
   <xacro:include filename="lidar.xacro" />
 </robot>
